File: audio.kicad_sch (KiCad schematic)
At the start: 19 parts, among them J13 Line Out, U7 PCM5102A

Commit message: Changed Line Out Connector
Changed Line Out Connector
Parts:
- J13: footprint Connector_Audio:Jack_3.5mm_CUI_SJ1-3514N_Horizontal -> Connector_Audio:Jack_3.5mm_CUI_SJ1-3524N_Horizontal
Changed lines of the file:
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@@
 			)
 		)
-		(property "Footprint" "Connector_Audio:Jack_3.5mm_CUI_SJ1-3514N_Horizontal"
+		(property "Footprint" "Connector_Audio:Jack_3.5mm_CUI_SJ1-3524N_Horizontal"
 			(at 233.68 66.04 0)
 			(effects

Commit message: Silkscreen fix
Fixed wrong silkcreen text for the DAC Voltage-Source. USB and +5V are flipped
Parts:
- D16, D17: footprint Diode_SMD:D_SOD-323 -> Diode_SMD:D_SOD-323_HandSoldering
Changed lines of the file:
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@@
 			)
 		)
-		(property "Footprint" "Diode_SMD:D_SOD-323"
+		(property "Footprint" "Diode_SMD:D_SOD-323_HandSoldering"
 			(at 205.74 73.66 0)
 			(effects
@@
 			)
 		)
-		(property "Footprint" "Diode_SMD:D_SOD-323"
+		(property "Footprint" "Diode_SMD:D_SOD-323_HandSoldering"
 			(at 187.96 73.66 0)
 			(effects
