File: BigCore.kicad_pcb (KiCad board)
At the start: 4 copper layers, 61 x 100 mm, 151 parts, among them J1 5V In, J10 Btn 3, J11 GND, J12 USB_C_Receptacle_USB2.0, J13 Line Out, J14 Servo 01, J15 Servo 02, J16 Servo 03, J17 Servo 04, J18 Servo 05, J19 Servo 06, J2 Vdrive In, J20 I2C, J22 WS2812, J3 JTAG, J4 DM3AT-SF-PEJM5, J5 Volume, J6 Btn 0, J7 RS485, J8 Btn 1, J9 Btn 2, Q1 SS8050-G, Q2 SS8050-G, SW1 Reset, SW2 Boot, SW3 Btn 0, SW4 Btn 1, SW5 Btn 2, SW6 Btn 3, U1 AP63203WU, U10 74AHCT1G17, U2 AP2112K-3.3, U3 ESP32-WROOM-32E, U4 ST3485EBDR, U5 USBLC6-2SC6, U6 CP2102N-Axx-xQFN24, U7 PCM5102A, U9 74AHCT1G17

Commit message: PCB Version Bump
-Bumped PCB to Version 1.1
Other:
- board text added: "Bottango BigCore v1.1"
- board text removed: "Bottango BigCore v1.0"
Changed lines of the file:
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@@
 		)
 	)
-	(gr_text "Bottango\nBigCore v1.0"
+	(gr_text "Bottango\nBigCore v1.1"
 		(at 84.6 200.4 0)
 		(layer "F.SilkS")

Commit message: Renamed PCB
Other:
- board text added: "Geistwerk // BigCore v1.1"
- board text removed: "Bottango BigCore v1.1"
Changed lines of the file:
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@@
 		)
 	)
-	(gr_text "Bottango\nBigCore v1.1"
+	(gr_text "Geistwerk //\nBigCore v1.1"
 		(at 84.6 200.4 0)
 		(layer "F.SilkS")

Commit message: Refreshed the BOM
Other:
- board text added: "Geistwerk //BigCore v1.1"
- board text removed: "Geistwerk // BigCore v1.1"
Changed lines of the file:
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@@
 		)
 	)
-	(gr_text "Geistwerk //\nBigCore v1.1"
+	(gr_text "Geistwerk\n//BigCore v1.1"
 		(at 84.6 200.4 0)
 		(layer "F.SilkS")
